File: first-microcontroller.kicad_sch (KiCad schematic)
At the start: 30 parts, among them J1 USB_C_Receptacle_USB2.0_14P, J2 ICSP Header, J3 Conn_02x13_Odd_Even, SW1 SW_RESET, U1 ATmega32U4-A, U2 USBLC6-2SC6, Y1 16Mhz

Commit message: fixed RST on ICSP header
Parts:
- removed R7: 10kΩ, symbol Device:R_Small_US
Connections:
- net at C2.2, C3.1, C4.1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: no longer J2.5 (Pin_5)
- net RST: now reaches R3.2, SW1.2, U1.13 (~{RESET})
- net RST: now also J2.5 (Pin_5)
Other:
- moved on the sheet: C2
Changed lines of the file:
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@@
 	(paper "A4")
 	(title_block
-		(date "2025-06-21")
-		(rev "v0.2")
+		(date "2025-06-22")
+		(rev "v0.3")
 		(comment 3 "ATMEGA32U4 breakout microcontroller")
 		(comment 4 "Author: Spencer Lommel")
@@
 	)
 	(junction
-		(at 162.56 96.52)
-		(diameter 0)
-		(color 0 0 0 0)
-	)
-	(junction
 		(at 67.31 96.52)
 		(diameter 0)
@@
 	)
 	(junction
-		(at 180.34 99.06)
-		(diameter 0)
-		(color 0 0 0 0)
-	)
-	(junction
 		(at 116.84 88.9)
 		(diameter 0)
@@
 	)
 	(junction
+		(at 180.34 96.52)
+		(diameter 0)
+		(color 0 0 0 0)
+	)
+	(junction
 		(at 137.16 39.37)
 		(diameter 0)
@@
 	)
 	(junction
-		(at 160.02 67.31)
-		(diameter 0)
-		(color 0 0 0 0)
-	)
-	(junction
 		(at 90.17 88.9)
 		(diameter 0)
@@
 	(wire
 		(pts
-			(xy 180.34 96.52) (xy 180.34 99.06)
-		)
-		(stroke
-			(width 0)
-			(type default)
-		)
-	)
-	(wire
-		(pts
 			(xy 118.11 116.84) (xy 90.17 116.84)
 		)
@@
 	(wire
 		(pts
-			(xy 160.02 96.52) (xy 160.02 67.31)
-		)
-		(stroke
-			(width 0)
-			(type default)
-		)
-	)
-	(wire
-		(pts
 			(xy 97.79 83.82) (xy 97.79 73.66)
 		)
@@
 	(wire
 		(pts
-			(xy 180.34 99.06) (xy 180.34 113.03)
+			(xy 180.34 96.52) (xy 180.34 113.03)
 		)
 		(stroke
@@
 	(wire
 		(pts
-			(xy 152.4 121.92) (xy 157.48 121.92)
-		)
-		(stroke
-			(width 0)
-			(type default)
-		)
-	)
-	(wire
-		(pts
 			(xy 144.78 58.42) (xy 144.78 62.23)
 		)
@@
 	(wire
 		(pts
-			(xy 162.56 96.52) (xy 162.56 121.92)
-		)
-		(stroke
-			(width 0)
-			(type default)
-		)
-	)
-	(wire
-		(pts
 			(xy 57.15 101.6) (xy 57.15 104.14)
 		)
@@
 	(wire
 		(pts
-			(xy 167.64 96.52) (xy 162.56 96.52)
-		)
-		(stroke
-			(width 0)
-			(type default)
-		)
-	)
-	(wire
-		(pts
-			(xy 162.56 96.52) (xy 160.02 96.52)
-		)
-		(stroke
-			(width 0)
-			(type default)
-		)
-	)
-	(wire
-		(pts
 			(xy 107.95 106.68) (xy 107.95 93.98)
 		)
@@
 	(wire
 		(pts
-			(xy 185.42 91.44) (xy 185.42 99.06)
+			(xy 185.42 91.44) (xy 185.42 96.52)
 		)
 		(stroke
@@
 		)
 	)
+	(label "RST"
+		(at 119.38 68.58 180)
+		(effects
+			(font
+				(size 1.27 1.27)
+			)
+			(justify right bottom)
+		)
+	)
 	(label "PB1"
 		(at 200.66 121.92 0)
@@
 		)
 	)
+	(label "RST"
+		(at 167.64 96.52 180)
+		(effects
+			(font
+				(size 1.27 1.27)
+			)
+			(justify right bottom)
+		)
+	)
 	(label "PD4"
 		(at 187.96 139.7 180)
@@
 	)
 	(symbol
-		(lib_id "Device:R_Small_US")
-		(at 160.02 121.92 90)
-		(unit 1)
-		(exclude_from_sim no)
-		(in_bom yes)
-		(on_board yes)
-		(dnp no)
-		(property "Reference" "R7"
-			(at 160.782 124.206 90)
-			(effects
-				(font
-					(size 1.27 1.27)
-				)
-			)
-		)
-		(property "Value" "10kΩ"
-			(at 160.782 126.238 90)
-			(effects
-				(font
-					(size 1.27 1.27)
-				)
-			)
-		)
-		(property "Footprint" ""
-			(at 160.02 121.92 0)
-			(effects
-				(font
-					(size 1.27 1.27)
-				)
-				(hide yes)
-			)
-		)
-		(property "Datasheet" "~"
-			(at 160.02 121.92 0)
-			(effects
-				(font
-					(size 1.27 1.27)
-				)
-				(hide yes)
-			)
-		)
-		(property "Description" "Resistor, small US symbol"
-			(at 160.02 121.92 0)
-			(effects
-				(font
-					(size 1.27 1.27)
-				)
-				(hide yes)
-			)
-		)
-		(pin "1"
-		)
-		(pin "2"
-		)
-		(instances
-			(project ""
-				(path "/7e81d9a1-b040-45be-bc17-b8565fca529e"
-					(reference "R7")
-					(unit 1)
-				)
-			)
-		)
-	)
-	(symbol
 		(lib_id "Device:C_Small")
-		(at 182.88 99.06 90)
+		(at 182.88 96.52 90)
 		(unit 1)
 		(exclude_from_sim no)
@@
 		(dnp no)
 		(property "Reference" "C2"
-			(at 183.642 101.6 90)
+			(at 183.642 99.06 90)
 			(effects
 				(font
@@
 		)
 		(property "Value" "0.1uF"
-			(at 184.404 103.378 90)
+			(at 184.404 100.838 90)
 			(effects
 				(font
@@
 		)
 		(property "Footprint" ""
-			(at 182.88 99.06 0)
+			(at 182.88 96.52 0)
 			(effects
 				(font
@@
 		)
 		(property "Datasheet" "~"
-			(at 182.88 99.06 0)
+			(at 182.88 96.52 0)
 			(effects
 				(font
@@
 		)
 		(property "Description" "Unpolarized capacitor, small symbol"
-			(at 182.88 99.06 0)
+			(at 182.88 96.52 0)
 			(effects
 				(font

Commit message: rev v0.4
Parts:
- TP2: value 5.5v TP -> 5v TP
Changed lines of the file:
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@@
 	(title_block
 		(date "2025-06-22")
-		(rev "v0.3")
+		(rev "v0.4")
 		(comment 3 "ATMEGA32U4 breakout microcontroller")
 		(comment 4 "Author: Spencer Lommel")
@@
 			)
 		)
-		(property "Value" "5.5v TP"
+		(property "Value" "5v TP"
 			(at 114.554 48.26 90)
 			(effects

Commit message: updated nets, fixed oscillator caps, better GND/VCC isolation
Parts:
- removed C11: 0.1uF, symbol Device:C_Small
- removed TP1: 3.3v TP, symbol Connector:TestPoint
- added J4: Conn_01x02, symbol Connector_Generic:Conn_01x02
Connections:
- net GND: now also J4.2 (Pin_2)
- net VCC: now reaches C2.2, C3.1, C4.1, C5.1, C6.1, FB1.1, J2.2 (Pin_2), R3.1, TP2.1, U1.14 (VCC), U1.2 (UVCC), U1.24 (AVCC), U1.34 (VCC), U1.44 (AVCC)
- net VBUS: now reaches C1.1, F1.2, FB1.2, U1.7 (VBUS), U2.5 (VBUS)
- net VBUS: no longer U1.42 (AREF)
- new net AREF: J4.1 (Pin_1), U1.42 (AREF)
Other:
- moved on the sheet: FB1, TP2
